Commit message: 为机器人添加虚拟部件，以贴合地面

File: test/chapt5/src/fishbot_description/urdf/fishbot/base.urdf.xacro (robot description, xacro)
@@ -2,4 +2,6 @@
 <robot xmlns:xacro="http://www.ros.org/wiki/xacro">
     <xacro:macro name="base_xacro" params="length radius">
+        <!-- 虚拟部件 -->
+        <link name="base_footprint"/>
         <!-- 机器人的身体部分 -->
         <link name="base_link">
@@ -19,4 +21,9 @@
             </visual>
         </link>
+        <joint name="joint_name" type="fixed">
+            <origin xyz="0.0 0.0 ${length / 2.0 + 0.032 - 0.001}" rpy="0.0 0.0 0.0"/>
+            <parent link="base_footprint"/>
+            <child link="base_link"/>
+        </joint>
     </xacro:macro>
 </robot>
