Commit message: 为机器人部件添加碰撞属性

File: test/chapt5/src/fishbot_description/urdf/fishbot/actuator/caster.urdf.xacro (robot description, xacro)
@@ -12,4 +12,13 @@
                 </material>
             </visual>
+            <collision>
+                <origin xyz="0.0 0.0 0.0" rpy="0.0 0.0 0.0"/>
+                <geometry>
+                    <sphere radius="0.016"/>
+                </geometry>
+                <material name="yellow">
+                    <color rgba="1.0 1.0 0.0 0.8"/>
+                </material>
+            </collision>
         </link>
         <!-- 机器人的关节，用于组合机器人的部件 -->

File: test/chapt5/src/fishbot_description/urdf/fishbot/actuator/wheel.urdf.xacro (robot description, xacro)
@@ -12,4 +12,13 @@
                 </material>
             </visual>
+            <collision>
+                <origin xyz="0.0 0.0 0.0" rpy="1.57079 0.0 0.0"/>
+                <geometry>
+                    <cylinder radius="0.032" length="0.04"/>
+                </geometry>
+                <material name="yellow">
+                    <color rgba="1.0 1.0 0.0 0.8"/>
+                </material>
+            </collision>
         </link>
         <!-- 机器人的关节，用于组合机器人的部件 -->

File: test/chapt5/src/fishbot_description/urdf/fishbot/base.urdf.xacro (robot description, xacro)
@@ -20,4 +20,17 @@
                 </material>
             </visual>
+            <collision>
+                <!-- 沿着自己几何中心的偏移和旋转量 -->
+                <origin xyz="0.0 0.0 0.0" rpy="0.0 0.0 0.0"/>
+                <!-- 几何形状 -->
+                <geometry>
+                    <!-- 圆柱体，半径：0.10m，高度：0.12m -->
+                    <cylinder radius="${radius}" length="${length}"/>
+                </geometry>
+                <!-- 材质颜色 -->
+                <material name="white">
+                    <color rgba="1.0 1.0 1.0 0.5"/>
+                </material>
+            </collision>
         </link>
         <joint name="joint_name" type="fixed">

File: test/chapt5/src/fishbot_description/urdf/fishbot/sensor/camera.urdf.xacro (robot description, xacro)
@@ -13,4 +13,13 @@
                 </material>
             </visual>
+            <collision>
+                <origin xyz="0.0 0.0 0.0" rpy="0.0 0.0 0.0"/>
+                <geometry>
+                    <box size="0.02 0.02 0.02"/>
+                </geometry>
+                <material name="black">
+                    <color rgba="0.0 0.0 0.0 0.5"/>
+                </material>
+            </collision>
         </link>
         <!-- 机器人的关节，用于组合机器人的部件 -->

File: test/chapt5/src/fishbot_description/urdf/fishbot/sensor/imu.urdf.xacro (robot description, xacro)
@@ -13,4 +13,13 @@
                 </material>
             </visual>
+            <collision>
+                <origin xyz="0.0 0.0 0.0" rpy="0.0 0.0 0.0"/>
+                <geometry>
+                    <box size="0.02 0.02 0.02"/>
+                </geometry>
+                <material name="black">
+                    <color rgba="0.0 0.0 0.0 0.5"/>
+                </material>
+            </collision>
         </link>
         <!-- 机器人的关节，用于组合机器人的部件 -->

File: test/chapt5/src/fishbot_description/urdf/fishbot/sensor/laser.urdf.xacro (robot description, xacro)
@@ -13,4 +13,13 @@
                 </material>
             </visual>
+            <collision>
+                <origin xyz="0.0 0.0 0.0" rpy="0.0 0.0 0.0"/>
+                <geometry>
+                    <cylinder radius="0.01" length="0.10"/>
+                </geometry>
+                <material name="black">
+                    <color rgba="0.0 0.0 0.0 1.0"/>
+                </material>
+            </collision>
         </link>
         <!-- 雷达 -->
@@ -25,4 +34,13 @@
                 </material>
             </visual>
+            <collision>
+                <origin xyz="0.0 0.0 0.0" rpy="0.0 0.0 0.0"/>
+                <geometry>
+                    <cylinder radius="0.02" length="0.02"/>
+                </geometry>
+                <material name="black">
+                    <color rgba="0.0 0.0 0.0 1.0"/>
+                </material>
+            </collision>
         </link>
         <!-- 机器人的关节，用于组合机器人的部件 -->

Commit message: 使用gazebo标签扩展urdf

File: test/chapt5/src/fishbot_description/urdf/fishbot/actuator/caster.urdf.xacro (robot description, xacro)
@@ -31,4 +31,10 @@
             <axis xyz="0 1 0"/>
         </joint>
+        <gazebo reference="${caster_name}_link">
+            <mu1 value="0.0"/>
+            <mu2 value="0.0"/>
+            <kp value="1000000000.0"/>
+            <kd value="1.0"/>
+        </gazebo>
     </xacro:macro>
 </robot>

File: test/chapt5/src/fishbot_description/urdf/fishbot/actuator/wheel.urdf.xacro (robot description, xacro)
@@ -31,4 +31,10 @@
             <axis xyz="0 1 0"/>
         </joint>
+        <gazebo reference="${wheel_name}_link">
+            <mu1 value="20.0"/>
+            <mu2 value="20.0"/>
+            <kp value="1000000000.0"/>
+            <kd value="1.0"/>
+        </gazebo>
     </xacro:macro>
 </robot>

File: test/chapt5/src/fishbot_description/urdf/fishbot/sensor/laser.urdf.xacro (robot description, xacro)
@@ -58,4 +58,10 @@
             <origin xyz="${xyz}" rpy="0.0 0.0 0.0"/>
         </joint>
+        <gazebo reference="laser_link">
+            <material>Gazebo/Black</material>
+        </gazebo>
+        <gazebo reference="laser_cylinder_link">
+            <material>Gazebo/Black</material>
+        </gazebo>
     </xacro:macro>
 </robot>
